File: HamRuler_v1/HamRuler_v1.sch (KiCad schematic (older format))
At the start: 13 parts, among them J1 Conn_01x03, Q1 BUK7M9R9-60EX, Q2 BUK7M9R9-60EX, U1 AT42QT1011-TSHR, U2 AT42QT1011-TSHR

Commit message: nightly
Parts:
- H1, H2: footprint Connector:Banana_Jack_1Pin -> Resources:Large Pad
Changed lines of the file:
@@
 F 0 "H1" V 3787 2453 50  0000 C CNN
 F 1 "MountingHole_Pad" V 3696 2453 50  0000 C CNN
-F 2 "Connector:Banana_Jack_1Pin" H 3550 2450 50  0001 C CNN
+F 2 "Resources:Large Pad" H 3550 2450 50  0001 C CNN
 F 3 "~" H 3550 2450 50  0001 C CNN
 	1    3550 2450
@@
 F 0 "H2" V 3787 3203 50  0000 C CNN
 F 1 "MountingHole_Pad" V 3696 3203 50  0000 C CNN
-F 2 "Connector:Banana_Jack_1Pin" H 3550 3200 50  0001 C CNN
+F 2 "Resources:Large Pad" H 3550 3200 50  0001 C CNN
 F 3 "~" H 3550 3200 50  0001 C CNN
 	1    3550 3200
